File: circuit-esp32-base.kicad_pcb (KiCad board)
At the start: 2 copper layers, 100 x 84 mm, 41 parts, among them J1 PWR, J10 PWM5, J11 PWM6, J12 IN, J13 IO_PWM, J14 DIO_PWM, J15 12VIO_1, J16 12VIO_2, J17 12VIO_3, J18 12VIO_4, J2 UART1, J3 UART2, J4 CAN_1, J5 CAN_2, J6 PWM1, J7 PWM2, J8 PWM3, J9 PWM4, SW1 RESET, SW2 SW_SPST, SW3 SW_SPST, SW4 SW_SPST, SW5 SW_SPST, U1 ESP32-DevKitC-32E, U2 MCP2542WFDxMF, U3 ULN2801A

Commit message: 基板サイズを変更。
Parts:
- moved   10.0 mm to (196.0, 80.0)
- moved   10.0 mm to (104.0, 80.0)
- moved G*** 3.35 mm to (110.5, 87.0)
Routing:
- net GND: vias 88 -> 79
Other:
- board size 100 x 84 mm -> 100 x 74 mm
