File: circuit-esp32-base.kicad_pcb (KiCad board)
At the start: 2 copper layers, 100 x 74 mm, 41 parts, among them J1 PWR, J10 PWM5, J11 PWM6, J12 IN, J13 IO_PWM, J14 DIO_PWM, J15 12VIO_1, J16 12VIO_2, J17 12VIO_3, J18 12VIO_4, J2 UART1, J3 UART2, J4 CAN_1, J5 CAN_2, J6 PWM1, J7 PWM2, J8 PWM3, J9 PWM4, SW1 RESET, SW2 SW_SPST, SW3 SW_SPST, SW4 SW_SPST, SW5 SW_SPST, U1 ESP32-DevKitC-32E, U2 MCP2542WFDxMF, U3 ULN2801A

Commit message: コンデンサの容量を変更。
Parts:
- C1, C2: value 10uF -> 0.1uF
Changed lines of the file:
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@@
 			)
 		)
-		(property "Value" "10uF"
+		(property "Value" "0.1uF"
 			(at 0 -1.43 0)
 			(layer "B.Fab")
@@
 			)
 		)
-		(property "Value" "10uF"
+		(property "Value" "0.1uF"
 			(at 0 -1.43 0)
 			(layer "B.Fab")

Commit message: 基板サイズを変更。
Parts:
- moved   4.00 mm to (104.0, 84.0)
- moved D1 3.53 mm to (195.7, 118.0)
- moved D2 3.53 mm to (195.7, 109.5)
- moved D3 3.53 mm to (195.7, 101.0)
- moved D4 3.53 mm to (195.7, 92.5)
- moved J15 3.53 mm to (187.5, 115.0)
- moved J16 3.53 mm to (187.5, 106.5)
- moved J17 3.53 mm to (187.5, 98.0)
- moved J18 3.53 mm to (187.7, 89.5)
- moved R1 3.53 mm to (195.7, 115.0)
- moved R2 3.53 mm to (195.7, 106.4)
- moved R3 3.53 mm to (195.7, 98.0)
- moved R4 3.53 mm to (195.7, 89.6)
- moved   3.50 mm to (196.0, 83.5)
- moved J10 3.50 mm to (158.5, 90.5)
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Routing:
- net +5V: track 144.1 -> 147.9 mm
- net 12VIO_4: track 56.7 -> 53.2 mm
- net 12VIO_3: track 44.0 -> 40.5 mm
- net 12VIO_2: track 30.8 -> 27.3 mm
- net 12VIO_1: track 16.4 -> 12.9 mm
- net IO_4: track 95.5 -> 92.0 mm
- net DIO_16: track 67.9 -> 64.4 mm
- net IO_12: track 108.0 -> 104.5 mm
- net DIO_5: track 72.5 -> 69.0 mm
- net DIO_21: track 45.5 -> 42.0 mm
- net DIO_17: track 62.6 -> 59.1 mm
- net IO_13: track 102.9 -> 99.7 mm
- net IO_14: track 105.7 -> 103.6 mm
- net +12V: track 100.8 -> 98.8 mm
- net DIO_18: track 60.9 -> 59.1 mm
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Other:
- board size 100 x 74 mm -> 100 x 70 mm
