File: circuit-esp32-base.kicad_pcb (KiCad board)
At the start: 2 copper layers, 100 x 70 mm, 41 parts, among them J1 PWR, J10 PWM5, J11 PWM6, J12 IN, J13 IO_PWM, J14 DIO_PWM, J15 12VIO_1, J16 12VIO_2, J17 12VIO_3, J18 12VIO_4, J2 UART1, J3 UART2, J4 CAN_1, J5 CAN_2, J6 PWM1, J7 PWM2, J8 PWM3, J9 PWM4, SW1 RESET, SW2 SW_SPST, SW3 SW_SPST, SW4 SW_SPST, SW5 SW_SPST, U1 ESP32-DevKitC-32E, U2 MCP2542WFDxMF, U3 ULN2801A

Commit message: 3.2ネジ穴の位置を修正。
Parts:
- moved   0.50 mm to (104.0, 83.5)
Routing:
- net GND: vias 79 -> 80
Changed lines of the file:
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@@
 	(footprint "circuit-esp32-base:holeφ3.2"
 		(layer "F.Cu")
-		(at 104 84)
+		(at 104 83.5)
 		(property "Reference" " "
 			(at 0 0.5 0)
@@
 	)
 	(via
+		(at 189 116.5)
+		(size 0.8)
+		(drill 0.4)
+		(layers "F.Cu" "B.Cu")
+		(free yes)
+		(net 2)
+	)
+	(via
 		(at 182 103)
 		(size 0.8)
@@
 	)
 	(segment
-		(start 135.060661 98)
-		(end 134.5 98)
+		(start 139.5 90)
+		(end 139.5 92.5)
 		(width 0.3)
 		(layer "F.Cu")
@@
 	)
 	(segment
-		(start 129 115)
-		(end 129 124)
+		(start 141.5 88)
+		(end 139.5 90)
 		(width 0.3)
 		(layer "F.Cu")
@@
 	)
 	(segment
-		(start 154.693898 139.693898)
-		(end 125.193898 139.693898)
+		(start 129 115)
+		(end 129 124)
 		(width 0.3)
 		(layer "F.Cu")
@@
 	)
 	(segment
-		(start 137.25 92.25)
-		(end 137.25 95.810661)
+		(start 154.693898 139.693898)
+		(end 125.193898 139.693898)
 		(width 0.3)
 		(layer "F.Cu")
@@
 	)
 	(segment
-		(start 141.5 88)
-		(end 137.25 92.25)
+		(start 139.5 92.5)
+		(end 137.25 94.75)
 		(width 0.3)
 		(layer "F.Cu")
@@
 		(width 0.3)
 		(layer "F.Cu")
+		(net 22)
+	)
+	(segment
+		(start 135.060661 98)
+		(end 134.5 98)
+		(width 0.3)
+		(layer "F.Cu")
+		(net 22)
+	)
+	(segment
+		(start 137.25 94.75)
+		(end 137.25 95.810661)
+		(width 0.3)
+		(layer "F.Cu")

Commit message: CANトランシーバのフットプリントを修正。 パスコンの位置を修正。 配線を修正。
Parts:
- C1, C2: moved to F.Cu
- J2, J3: footprint ms0503:DF1B-4P-2.5DSA -> circuit-esp32-base:DF1B-4P-2.5DSA
- U2: footprint Package_DFN_QFN:DFN-8-1EP_3x3mm_P0.65mm_EP1.55x2.4mm -> Package_DFN_QFN:DFN-8-1EP_6x5mm_P1.27mm_EP2x2mm
- moved C1 2.83 mm to (159.5, 109.5), turned to -90 degrees
- moved C2 1.58 mm to (152.0, 105.0), turned to 90 degrees
Connections:
- SW1 pad 2: unconnected-(SW1-Pad2) -> GND
Routing:
- net GND: track 5.42 -> 0.00 mm, vias 80 -> 79
- net Net-(U1-IO23): track 9.04 -> 7.41 mm
- net Net-(U1-IO22): track 9.02 -> 7.43 mm
- net CAN_P: track 19.8 -> 18.6 mm
- net CAN_N: track 20.6 -> 19.5 mm
- net +3V3: track 52.6 -> 53.7 mm
Other:
- board text added: "v2"

Commit message: タクトスイッチの向きを修正。 直角配線を撲滅。 上部GPIO3ピンコネクタの向きを修正。
Parts:
- moved J10 5.00 mm to (158.5, 85.5), turned to -90 degrees
- moved J11 5.00 mm to (167.0, 85.5), turned to -90 degrees
- moved J6 5.00 mm to (124.5, 85.5), turned to -90 degrees
- moved J7 5.00 mm to (133.1, 85.5), turned to -90 degrees
- moved J8 5.00 mm to (141.5, 85.5), turned to -90 degrees
- moved J9 5.00 mm to (150.0, 85.5), turned to -90 degrees
- moved J18 0.15 mm to (187.5, 89.5)
Connections:
- J10 pad 1: DIO_19 -> GND
- J10 pad 3: GND -> DIO_19
- J11 pad 1: DIO_21 -> GND
- J11 pad 3: GND -> DIO_21
- J6 pad 1: DIO_5 -> GND
- J6 pad 3: GND -> DIO_5
- J7 pad 1: DIO_16 -> GND
- J7 pad 3: GND -> DIO_16
- J8 pad 1: DIO_17 -> GND
- J8 pad 3: GND -> DIO_17
- J9 pad 1: DIO_18 -> GND
- J9 pad 3: GND -> DIO_18
- SW2 pad ~1: (no net) -> GND
- SW2 pad ~2: (no net) -> GND
- SW3 pad ~1: (no net) -> GND
- SW3 pad ~2: (no net) -> GND
- SW4 pad ~1: (no net) -> GND
- SW4 pad ~2: (no net) -> GND
- SW5 pad ~1: (no net) -> GND
- SW5 pad ~2: (no net) -> GND
Routing:
- net +12V: track 98.8 -> 117.2 mm
- net +5V: track 147.7 -> 155.4 mm
Other:
- board text added: "v3"
- board text removed: "v2"
