File: circuit-esp32-base.kicad_sch (KiCad schematic)
At the start: 36 parts, among them J1 PWR, J10 PWM5, J11 PWM6, J12 IN, J13 IO_PWM, J14 DIO_PWM, J15 12VIO_1, J16 12VIO_2, J17 12VIO_3, J18 12VIO_4, J2 UART1, J3 UART2, J4 CAN_1, J5 CAN_2, J6 PWM1, J7 PWM2, J8 PWM3, J9 PWM4, SW1 RESET, SW2 SW_SPST, SW3 SW_SPST, SW4 SW_SPST, SW5 SW_SPST, U1 ESP32-DevKitC-32E, U2 MCP2542WFDxMF, U3 ULN2801A

Commit message: コンデンサの容量を変更。
Parts:
- C1, C2: value 10uF -> 0.1uF
Changed lines of the file:
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@@
 			)
 		)
-		(property "Value" "10uF"
+		(property "Value" "0.1uF"
 			(at 99.822 38.1 0)
 			(effects
@@
 			)
 		)
-		(property "Value" "10uF"
+		(property "Value" "0.1uF"
 			(at 124.46 38.0999 0)
 			(effects

Commit message: CANトランシーバのフットプリントを修正。 パスコンの位置を修正。 配線を修正。
Parts:
- J12: footprint ms0503:4pin -> circuit-esp32-base:4pin
- J13: footprint ms0503:8pin -> circuit-esp32-base:8pin
- J14: footprint ms0503:6pin -> circuit-esp32-base:6pin
- J2, J3: footprint ms0503:DF1B-4P-2.5DSA -> circuit-esp32-base:DF1B-4P-2.5DSA
- SW1: footprint mecha:tact -> circuit-esp32-base:tact
- SW2, SW3, SW4, SW5: footprint mecha:toggle_1-2 -> circuit-esp32-base:toggle_1-2
- U1: footprint ms0503:ESP32-DevKitC-32E -> circuit-esp32-base:ESP32-DevKitC-32E
- U2: footprint Package_DFN_QFN:DFN-8-1EP_3x3mm_P0.65mm_EP1.55x2.4mm -> Package_DFN_QFN:DFN-8-1EP_6x5mm_P1.27mm_EP2x2mm
Connections:
- net GND: now also SW1.2
- no-connect marks 22 -> 21
Changed lines of the file:
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@@
 	)
 	(junction
+		(at 34.29 52.07)
+		(diameter 0)
+		(color 0 0 0 0)
+	)
+	(junction
 		(at 165.1 100.33)
 		(diameter 0)
@@
 	)
 	(no_connect
-		(at 36.83 52.07)
-	)
-	(no_connect
 		(at 228.6 57.15)
 	)
@@
 	(wire
 		(pts
+			(xy 34.29 52.07) (xy 34.29 54.61)
+		)
+		(stroke
+			(width 0)
+			(type default)
+		)
+	)
+	(wire
+		(pts
 			(xy 160.02 157.48) (xy 160.02 160.02)
 		)
@@
 	(wire
 		(pts
+			(xy 34.29 52.07) (xy 36.83 52.07)
+		)
+		(stroke
+			(width 0)
+			(type default)
+		)
+	)
+	(wire
+		(pts
 			(xy 49.53 132.08) (xy 49.53 129.54)
 		)
@@
 	(wire
 		(pts
-			(xy 34.29 49.53) (xy 34.29 54.61)
+			(xy 34.29 49.53) (xy 34.29 52.07)
 		)
 		(stroke
@@
 			)
 		)
-		(property "Footprint" "ms0503:6pin"
+		(property "Footprint" "circuit-esp32-base:6pin"
 			(at 152.4 100.33 0)
 			(effects
@@
 			)
 		)
-		(property "Footprint" "ms0503:DF1B-4P-2.5DSA"
+		(property "Footprint" "circuit-esp32-base:DF1B-4P-2.5DSA"
 			(at 74.93 134.62 0)
 			(effects
@@
 			)
 		)
-		(property "Footprint" "ms0503:8pin"
+		(property "Footprint" "circuit-esp32-base:8pin"
 			(at 152.4 57.15 0)
 			(effects
@@
 			)
 		)
-		(property "Footprint" "mecha:toggle_1-2"
+		(property "Footprint" "circuit-esp32-base:toggle_1-2"
 			(at 193.04 64.77 0)
 			(effects
@@
 			)
 		)
-		(property "Footprint" "mecha:toggle_1-2"
+		(property "Footprint" "circuit-esp32-base:toggle_1-2"
 			(at 193.04 95.25 0)
 			(effects
@@
 			)
 		)
-		(property "Footprint" "ms0503:DF1B-4P-2.5DSA"
+		(property "Footprint" "circuit-esp32-base:DF1B-4P-2.5DSA"
 			(at 41.91 134.62 0)
 			(effects
@@
 			)
 		)
-		(property "Footprint" "Package_DFN_QFN:DFN-8-1EP_3x3mm_P0.65mm_EP1.55x2.4mm"
+		(property "Footprint" "Package_DFN_QFN:DFN-8-1EP_6x5mm_P1.27mm_EP2x2mm"
 			(at 115.57 67.31 0)
 			(effects
@@
 			)
 		)
-		(property "Footprint" "ms0503:ESP32-DevKitC-32E"
+		(property "Footprint" "circuit-esp32-base:ESP32-DevKitC-32E"
 			(at 69.85 32.512 0)
 			(effects
@@
 			)
 		)
-		(property "Footprint" "ms0503:4pin"
+		(property "Footprint" "circuit-esp32-base:4pin"
 			(at 107.95 182.88 0)
 			(effects
@@
 			)
 		)
-		(property "Footprint" "mecha:toggle_1-2"
+		(property "Footprint" "circuit-esp32-base:toggle_1-2"
 			(at 193.04 49.53 0)
 			(effects
@@
 			)
 		)
-		(property "Footprint" "mecha:toggle_1-2"
+		(property "Footprint" "circuit-esp32-base:toggle_1-2"
 			(at 193.04 80.01 0)
 			(effects
@@
 			)
 		)
-		(property "Footprint" "mecha:tact"
+		(property "Footprint" "circuit-esp32-base:tact"
 			(at 41.91 44.45 0)
 			(effects

Commit message: タクトスイッチの向きを修正。 直角配線を撲滅。 上部GPIO3ピンコネクタの向きを修正。
Connections:
- net DIO_16: now also J7.3 (Pin_3); no longer J7.1 (Pin_1)
- net DIO_17: now also J8.3 (Pin_3); no longer J8.1 (Pin_1)
- net DIO_18: now also J9.3 (Pin_3); no longer J9.1 (Pin_1)
- net DIO_19: now also J10.3 (Pin_3); no longer J10.1 (Pin_1)
- net DIO_21: now also J11.3 (Pin_3); no longer J11.1 (Pin_1)
- net DIO_5: now also J6.3 (Pin_3); no longer J6.1 (Pin_1)
- net GND: now also J10.1 (Pin_1), J11.1 (Pin_1), J6.1 (Pin_1), J7.1 (Pin_1), J8.1 (Pin_1), J9.1 (Pin_1); no longer J10.3 (Pin_3), J11.3 (Pin_3), J6.3 (Pin_3), J7.3 (Pin_3), J8.3 (Pin_3), J9.3 (Pin_3)
